File: Master/IoTMasterPCB/Flash.sch (KiCad schematic (older format))
At the start: 2 parts

Commit message: Finished RFID module sans antenna footprint. Added KSZ8081MNX and hierarchial connections.
Changed lines of the file:
@@
 Wire Notes Line
 	7150 4300 5100 4300
-Text Notes 5100 4400 0    50   ~ 0
+Text Notes 5100 2700 0    50   ~ 0
 32 Mbit NOR Flash
 $EndSCHEMATC

Commit message: Finished RFID and Ethernet circuits.
Parts:
- C64: renamed from C?; footprint (none) -> Capacitor_SMD:C_0603_1608Metric
- gave numbers to parts that had none: 1
Changed lines of the file:
@@
 $EndDescr
 $Comp
-L Memory_Flash:W25Q32JVSS U?
+L Memory_Flash:W25Q32JVSS U7
 U 1 1 5FCEBC9A
 P 6150 3650
-F 0 "U?" H 6400 3250 50  0000 C CNN
+F 0 "U7" H 6400 3250 50  0000 C CNN
 F 1 "W25Q32JVSS" H 6600 3150 50  0000 C CNN
 F 2 "Package_SO:SOIC-8_5.23x5.23mm_P1.27mm" H 6150 3650 50  0001 C CNN
@@
 $EndComp
 $Comp
-L power:+3V3 #PWR?
+L power:+3V3 #PWR0173
 U 1 1 5FCEC418
 P 6150 2950
-F 0 "#PWR?" H 6150 2800 50  0001 C CNN
+F 0 "#PWR0173" H 6150 2800 50  0001 C CNN
 F 1 "+3V3" H 6165 3123 50  0000 C CNN
 F 2 "" H 6150 2950 50  0001 C CNN
@@
 $EndComp
 $Comp
-L Device:C C?
+L Device:C C64
 U 1 1 5FCECA90
 P 6400 3100
-F 0 "C?" V 6200 3200 50  0000 C CNN
+F 0 "C64" V 6200 3200 50  0000 C CNN
 F 1 "100 nF" V 6300 3300 50  0000 C CNN
-F 2 "" H 6438 2950 50  0001 C CNN
+F 2 "Capacitor_SMD:C_0603_1608Metric" H 6438 2950 50  0001 C CNN
 F 3 "~" H 6400 3100 50  0001 C CNN
 	1    6400 3100
@@
 Connection ~ 6150 3100
 $Comp
-L power:GND #PWR?
+L power:GND #PWR0174
 U 1 1 5FCED53D
 P 6600 3150
-F 0 "#PWR?" H 6600 2900 50  0001 C CNN
+F 0 "#PWR0174" H 6600 2900 50  0001 C CNN
 F 1 "GND" H 6600 3000 50  0000 C CNN
 F 2 "" H 6600 3150 50  0001 C CNN
@@
 	6600 3100 6600 3150
 $Comp
-L power:GND #PWR?
+L power:GND #PWR0175
 U 1 1 5FCEDBA2
 P 6150 4100
-F 0 "#PWR?" H 6150 3850 50  0001 C CNN
+F 0 "#PWR0175" H 6150 3850 50  0001 C CNN
 F 1 "GND" H 6150 3950 50  0000 C CNN
 F 2 "" H 6150 4100 50  0001 C CNN
