File: Master/IoTMasterPCB/PowerSupply.sch (KiCad schematic (older format))
At the start: 8 parts, among them J2 10118194-0001LF, U2 MYRGP330100B21RA

Commit message: Placed STM32 on Master PCB. Corrected I2C naming.
Connections:
- net +5V: no longer D1.1 (K)
- net GND: no longer D1.2 (A)
- net GND1: now also D1.2 (A)
- net at FB1.2, J2.1 (VBUS): now also D1.1 (K)
Other:
- moved on the sheet: C26, D1
Changed lines of the file:
@@
 L Device:C C26
 U 1 1 5FCBC1DA
-P 1450 3250
-F 0 "C26" H 1200 3300 50  0000 L CNN
-F 1 "4.7 µF" H 1100 3200 50  0000 L CNN
-F 2 "Capacitor_SMD:C_0805_2012Metric" H 1488 3100 50  0001 C CNN
-F 3 "~" H 1450 3250 50  0001 C CNN
-	1    1450 3250
+P 1600 3250
+F 0 "C26" H 1350 3300 50  0000 L CNN
+F 1 "4.7 µF" H 1250 3200 50  0000 L CNN
+F 2 "Capacitor_SMD:C_0805_2012Metric" H 1638 3100 50  0001 C CNN
+F 3 "~" H 1600 3250 50  0001 C CNN
+	1    1600 3250
 	1    0    0    -1
 $EndComp
-Wire Wire Line
-	1350 3100 1450 3100
 Wire Wire Line
 	1800 3100 1800 3250
 Wire Wire Line
 	1800 3250 1950 3250
-Wire Wire Line
-	1350 3400 1450 3400
 $Comp
 L power:GND #PWR0122
@@
 L Device:D_Zener_Small D1
 U 1 1 5FCF858A
-P 1600 3250
-F 0 "D1" V 1646 3180 50  0000 R CNN
-F 1 "5.6 V" V 1555 3180 50  0000 R CNN
-F 2 "Diode_SMD:D_MiniMELF" V 1600 3250 50  0001 C CNN
-F 3 "https://www.mouser.dk/ProductDetail/Rectron/ZMM5232B?qs=0s%252B5lLZkUHrTZgVrCvE0jA%3D%3D" V 1600 3250 50  0001 C CNN
-	1    1600 3250
+P 2200 2050
+F 0 "D1" H 2250 1950 50  0000 R CNN
+F 1 "5.6 V" H 2300 1850 50  0000 R CNN
+F 2 "Diode_SMD:D_MiniMELF" V 2200 2050 50  0001 C CNN
+F 3 "https://www.mouser.dk/ProductDetail/Rectron/ZMM5232B?qs=0s%252B5lLZkUHrTZgVrCvE0jA%3D%3D" V 2200 2050 50  0001 C CNN
+	1    2200 2050
+	1    0    0    -1
+$EndComp
+Connection ~ 1600 3100
+Wire Wire Line
+	1600 3100 1800 3100
+Connection ~ 1600 3400
+Wire Wire Line
+	1600 3400 1900 3400
+Wire Wire Line
+	1350 3400 1600 3400
+Wire Wire Line
+	1350 3100 1600 3100
+Wire Wire Line
+	1750 1750 1750 2050
+Wire Wire Line
+	1750 2050 2100 2050
+Connection ~ 1750 1750
+$Comp
+L power:GND1 #PWR?
+U 1 1 5FE5082A
+P 2350 2050
+F 0 "#PWR?" H 2350 1800 50  0001 C CNN
+F 1 "GND1" V 2350 1850 50  0000 C CNN
+F 2 "" H 2350 2050 50  0001 C CNN
+F 3 "" H 2350 2050 50  0001 C CNN
+	1    2350 2050
 	0    -1   -1   0
 $EndComp
 Wire Wire Line
-	1450 3100 1600 3100
-Connection ~ 1450 3100
-Wire Wire Line
-	1600 3150 1600 3100
-Connection ~ 1600 3100
-Wire Wire Line
-	1600 3100 1800 3100
-Wire Wire Line
-	1600 3350 1600 3400
-Wire Wire Line
-	1600 3400 1900 3400
-Wire Wire Line
-	1600 3400 1450 3400
-Connection ~ 1600 3400
-Connection ~ 1450 3400
+	2300 2050 2350 2050
 $EndSCHEMATC
